File: board/fan-switch.kicad_pcb (KiCad board)
At the start: 2 copper layers, 50 x 35 mm, 23 parts, among them J1 M+, J2 M-, J3 12V, J4 GND, Q1 BXT420N03M, U1 LM1117-3.3, U2 ESP-12, X1 ESP-PROG

Commit message: WIP
Parts:
- removed C4: 47u, Capacitor_SMD:C_0805_2012Metric_Pad1.18x1.45mm_HandSolder
- removed C5, C6: 100n, Capacitor_SMD:C_0805_2012Metric_Pad1.18x1.45mm_HandSolder
- removed R4, R5, R6, R7: 10k, Resistor_SMD:R_0805_2012Metric_Pad1.20x1.40mm_HandSolder
- removed X1: ESP-PROG, Drake:Micro-Match-FOB-6
- added J5: PROG, Connector_PinHeader_2.54mm:PinHeader_1x03_P2.54mm_Vertical, F.Cu at (143.5, 111.0)
- C2: value 10u -> 47u
- D2: value BAT54C -> LED; footprint Package_TO_SOT_SMD:SOT-23_Handsoldering -> LED_SMD:LED_0805_2012Metric_Pad1.15x1.40mm_HandSolder
- J1: value M+ -> 12V
- J2: value M- -> GND
- J3: value 12V -> M+
- J4: value GND -> M-
- Q1: footprint Package_TO_SOT_SMD:SOT-23_Handsoldering -> Package_TO_SOT_SMD:SOT-23
- R3: value 10k -> 270R
- U1: value LM1117-3.3 -> ESP32-C3-WROOM-02; footprint Package_TO_SOT_SMD:SOT-223-3_TabPin2 -> Espressif:ESP32-C3-WROOM-02
- U2: value ESP-12 -> LM1117-3.3; footprint Drake:ESP-12 -> Package_TO_SOT_SMD:SOT-223-3_TabPin2
- moved J4 38.5 mm to (144.0, 106.0)
- moved J3 38.3 mm to (144.0, 100.0)
- moved D2 38.1 mm to (111.0, 100.0), turned to -90 degrees
- moved Q1 36.2 mm to (143.0, 117.0)
- moved D1 30.0 mm to (139.0, 103.0), turned to -90 degrees
- moved R3 28.3 mm to (111.0, 104.0), turned to 90 degrees
- moved J1 27.7 mm to (106.0, 100.0)
- moved C2 26.1 mm to (114.0, 118.0)
- moved R1 23.1 mm to (137.0, 115.0), turned to 0 degrees
- moved U1 19.7 mm to (125.0, 102.0)
- moved R2 18.1 mm to (137.0, 119.0)
- moved U2 17.5 mm to (108.0, 118.0), turned to -90 degrees
- moved C3 12.6 mm to (117.0, 118.0), turned to 90 degrees
- moved J2 9.51 mm to (106.0, 106.0)
- moved C1 2.83 mm to (108.0, 111.0)
Connections:
- C2 pad 1: /3V3-LOCAL -> +3V3
- C3 pad 1: VCC -> +3V3
- D2 pad 1: /3V3-LOCAL -> GND
- D2 pad 2: /3V3-PROG -> Net-(D2-A)
- J2 pad 1: Net-(D1-A) -> GND
- J4 pad 1: GND -> Net-(D1-A)
- R3 pad 1: /GPIO0 -> /LED
- R3 pad 2: VCC -> Net-(D2-A)
- U1 pad 1: GND -> +3V3
- U1 pad 2: /3V3-LOCAL -> +3V3
- U1 pad 3: +12V -> /LED
- U2 pad 1: /RESET -> GND
- U2 pad 2: unconnected-(U2-ADC) -> +3V3
- U2 pad 3: /EN -> +12V
Routing:
- net VCC: track 55.4 -> 0.00 mm
- net /RESET: track 42.0 -> 0.00 mm, vias 2 -> 0
- net GND: track 29.4 -> 0.00 mm, vias 10 -> 0
- net /3V3-PROG: track 25.8 -> 0.00 mm, vias 2 -> 0
- net +3V3: track 0.00 -> 21.5 mm, vias 0 -> 6
- net Net-(Q1-G): track 21.8 -> 4.50 mm
- net /USB_D+: track 0.00 -> 15.1 mm
- net /3V3-LOCAL: track 13.9 -> 0.00 mm
- net /GPIO0: track 12.9 -> 0.00 mm
- net +12V: track 56.4 -> 68.4 mm
- net /RX: track 10.1 -> 0.00 mm
- net /USB_D-: track 0.00 -> 8.53 mm
- net /LED: track 0.00 -> 8.14 mm
- net Net-(D1-A): track 10.1 -> 18.2 mm
- net /GPIO15: track 6.20 -> 0.00 mm
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- added copper zone on B.Cu, net +3V3
- added copper zone on F.Cu, net GND
- removed copper zone on B.Cu, net GND
